File: ADC & REF.sch (KiCad schematic (older format))
At the start: 16 parts

Commit message: v1.0
Connections:
- net labels added: ADC_SPI1_CS0, ADC_SPI1_MOSI_ADC_CH_SEL, ADC_SPI1_SCLK, ADC_SPI1_SDO
- net labels removed: ADC_CH_SEL, SPI1_CS, SPI1_SCLK, SPI1_SDO
- wire segments 58 -> 77
Other:
- note added: "DVDD ? Wofür ? brauchen wir es?\nCH_SEL mit was gleichzeitig steuern ??\n"
- note removed: "DVDD ? Wofür ? brauchen wir es?\nCH_SEL mit was gleichzeitig steuern ??"
- moved on the sheet: C?, R?, U?

Commit message: Stand 10.03
Connections:
- net Vref: now reaches C?.1, C?.1, U?.2 (OUT), U?.3 (REF)
Changed lines of the file:
@@
 	6805 3110 6805 3015
 Wire Wire Line
-	6645 3015 6805 3015
-Wire Wire Line
-	6805 3015 6950 3015
+	6645 3015 6950 3015
 Wire Wire Line
 	7155 3005 7070 3005
@@
 	7155 2590 6515 2590
 Wire Wire Line
-	5825 4960 7485 4960
-Wire Wire Line
-	7485 4960 7655 4960
+	5825 4960 7655 4960
 Wire Wire Line
 	7485 5255 7485 5215
 Wire Wire Line
-	8355 3405 8480 3405
-Wire Wire Line
-	8480 3405 8680 3405
-Wire Wire Line
-	8680 3405 9135 3405
+	8355 3405 9135 3405
 Wire Wire Line
 	8680 3480 8680 3405
@@
 	7050 3205 7050 3330
 Wire Wire Line
-	7050 3330 6805 3330
-Wire Wire Line
-	6805 3330 6695 3330
+	7050 3330 6695 3330
 Wire Wire Line
 	6805 3310 6805 3330
@@
 	7030 3505 7030 3745
 Wire Wire Line
-	7030 3745 6800 3745
-Wire Wire Line
-	6800 3745 6655 3745
+	7030 3745 6655 3745
 Wire Wire Line
 	6805 3720 6805 3745
@@
 	6905 3405 6905 3505
 Wire Wire Line
-	6905 3505 6805 3505
-Wire Wire Line
-	6805 3505 6700 3505
+	6905 3505 6700 3505
 Wire Wire Line
 	6805 3520 6805 3505
@@
 	8680 3705 8680 3680
 Wire Wire Line
-	8355 3705 8480 3705
+	8355 3705 8680 3705
 Wire Wire Line
-	8480 3705 8680 3705
-Wire Wire Line
-	8480 4205 8480 3705
-Wire Wire Line
-	8480 3705 8480 3675
+	8480 4205 8480 3675
 Connection ~ 8480 3705
 Wire Wire Line
 	9135 3405 9135 4960
 Wire Wire Line
-	9135 4960 8455 4960
+	8455 4960 9220 4960
 Wire Wire Line
-	6810 4205 7040 4205
+	6810 4205 8480 4205
 Wire Wire Line
-	7040 4205 7755 4205
-Wire Wire Line
-	7755 4205 8480 4205
-Wire Wire Line
-	7755 2240 7755 2395
-Wire Wire Line
-	7755 2395 7755 2530
-Wire Wire Line
-	7755 2530 7755 2605
+	7755 2240 7755 2605
 Wire Wire Line
 	8055 5350 8055 5310
@@
 Connection ~ 7040 4205
 Wire Wire Line
-	5825 3905 6810 3905
-Wire Wire Line
-	6810 3905 7040 3905
-Wire Wire Line
-	7040 3905 7155 3905
+	5825 3905 7155 3905
 Wire Wire Line
 	7040 3905 7040 3985
@@
 	7755 2395 5825 2395
 Wire Wire Line
-	5825 2395 5825 3905
-Wire Wire Line
-	5825 3905 5825 4960
+	5825 2395 5825 4960
 Connection ~ 7755 2395
 Wire Wire Line
@@
 Wire Wire Line
 	8075 2530 8025 2530
+Text GLabel 9220 4960 2    60   Input ~ 0
+Vref
+Connection ~ 9135 4960
 $EndSCHEMATC

Commit message: schematics ==> Check (exept BW) Layout started
Parts:
- C10, C11, C12, C13, C14, C15, C16, C17: renamed from C?; footprint (none) -> Capacitors_SMD:C_0603
- R10, R5, R6, R7, R8, R9: renamed from R?; footprint (none) -> Resistors_SMD:R_0603
- U4: renamed from U?; footprint (none) -> Housings_DFN_QFN:QFN-16-1EP_3x3mm_Pitch0.5mm
- U5: renamed from U?; footprint TO_SOT_Packages_SMD:SOT-23 -> .pretty:SOT-23
Changed lines of the file:
@@
 ADC_2
 $Comp
-L R_Small R?
+L R_Small R5
 U 1 1 58B84E5D
 P 6545 3015
-F 0 "R?" H 6575 3035 50  0000 L CNN
+F 0 "R5" H 6575 3035 50  0000 L CNN
 F 1 "5" H 6575 2975 50  0000 L CNN
-F 2 "" H 6545 3015 50  0000 C CNN
+F 2 "Resistors_SMD:R_0603" H 6545 3015 50  0001 C CNN
 F 3 "" H 6545 3015 50  0000 C CNN
 	1    6545 3015
@@
 $EndComp
 $Comp
-L R_Small R?
+L R_Small R6
 U 1 1 58B84F1C
 P 6555 3745
-F 0 "R?" H 6585 3765 50  0000 L CNN
+F 0 "R6" H 6585 3765 50  0000 L CNN
 F 1 "5" H 6585 3705 50  0000 L CNN
-F 2 "" H 6555 3745 50  0000 C CNN
+F 2 "Resistors_SMD:R_0603" H 6555 3745 50  0001 C CNN
 F 3 "" H 6555 3745 50  0000 C CNN
 	1    6555 3745
@@
 $EndComp
 $Comp
-L C_Small C?
+L C_Small C11
 U 1 1 58B84FEC
 P 6805 3620
-F 0 "C?" H 6815 3690 50  0000 L CNN
+F 0 "C11" H 6815 3690 50  0000 L CNN
 F 1 "470p" H 6815 3540 50  0000 L CNN
-F 2 "" H 6805 3620 50  0000 C CNN
+F 2 "Capacitors_SMD:C_0603" H 6805 3620 50  0001 C CNN
 F 3 "" H 6805 3620 50  0000 C CNN
 	1    6805 3620
@@
 $EndComp
 $Comp
-L R_Small R?
+L R_Small R8
 U 1 1 58B85861
 P 6600 3505
-F 0 "R?" H 6630 3525 50  0000 L CNN
+F 0 "R8" H 6630 3525 50  0000 L CNN
 F 1 "5" H 6630 3465 50  0000 L CNN
-F 2 "" H 6600 3505 50  0000 C CNN
+F 2 "Resistors_SMD:R_0603" H 6600 3505 50  0001 C CNN
 F 3 "" H 6600 3505 50  0000 C CNN
 	1    6600 3505
@@
 $EndComp
 $Comp
-L GND #PWR?
+L GND #PWR013
 U 1 1 58B858FF
 P 6430 3505
-F 0 "#PWR?" H 6430 3255 50  0001 C CNN
+F 0 "#PWR013" H 6430 3255 50  0001 C CNN
 F 1 "GND" H 6430 3355 50  0000 C CNN
 F 2 "" H 6430 3505 50  0000 C CNN
@@
 $EndComp
 $Comp
-L R_Small R?
+L R_Small R7
 U 1 1 58B85D6C
 P 6595 3330
-F 0 "R?" H 6625 3350 50  0000 L CNN
+F 0 "R7" H 6625 3350 50  0000 L CNN
 F 1 "5" H 6625 3290 50  0000 L CNN
-F 2 "" H 6595 3330 50  0000 C CNN
+F 2 "Resistors_SMD:R_0603" H 6595 3330 50  0001 C CNN
 F 3 "" H 6595 3330 50  0000 C CNN
 	1    6595 3330
@@
 $EndComp
 $Comp
-L GND #PWR?
+L GND #PWR014
 U 1 1 58B85D72
 P 6425 3330
-F 0 "#PWR?" H 6425 3080 50  0001 C CNN
+F 0 "#PWR014" H 6425 3080 50  0001 C CNN
 F 1 "GND" H 6425 3180 50  0000 C CNN
 F 2 "" H 6425 3330 50  0000 C CNN
@@
 ADC_SPI1_CS0
 $Comp
-L REF3030 U?
+L REF3030 U5
 U 1 1 58B981ED
 P 8055 5010
-F 0 "U?" H 7855 5210 50  0000 C CNN
+F 0 "U5" H 7855 5210 50  0000 C CNN
 F 1 "REF3030" H 8005 5210 50  0000 L CNN
-F 2 "TO_SOT_Packages_SMD:SOT-23" H 8055 5110 50  0001 C CIN
+F 2 ".pretty:SOT-23" H 8055 5110 50  0001 C CIN
 F 3 "" H 8055 5010 50  0000 C CNN
 	1    8055 5010
@@
 $EndComp
 $Comp
-L C_Small C?
+L C_Small C14
 U 1 1 58B98B75
 P 7485 5115
-F 0 "C?" H 7495 5185 50  0000 L CNN
+F 0 "C14" H 7495 5185 50  0000 L CNN
 F 1 "470n" H 7495 5035 50  0000 L CNN
-F 2 "" H 7485 5115 50  0000 C CNN
+F 2 "Capacitors_SMD:C_0603" H 7485 5115 50  0001 C CNN
 F 3 "" H 7485 5115 50  0000 C CNN
 	1    7485 5115
@@
 $EndComp
 $Comp
-L GND #PWR?
+L GND #PWR015
 U 1 1 58B98FCA
 P 7485 5255
-F 0 "#PWR?" H 7485 5005 50  0001 C CNN
+F 0 "#PWR015" H 7485 5005 50  0001 C CNN
 F 1 "GND" H 7485 5105 50  0000 C CNN
 F 2 "" H 7485 5255 50  0000 C CNN
@@
 $EndComp
 $Comp
-L R_Small R?
+L R_Small R9
 U 1 1 58B99682
 P 7755 2140
-F 0 "R?" H 7785 2160 50  0000 L CNN
+F 0 "R9" H 7785 2160 50  0000 L CNN
 F 1 "5" H 7785 2100 50  0000 L CNN
-F 2 "" H 7755 2140 50  0000 C CNN
+F 2 "Resistors_SMD:R_0603" H 7755 2140 50  0001 C CNN
 F 3 "" H 7755 2140 50  0000 C CNN
 	1    7755 2140
@@
 $EndComp
 $Comp
-L C_Small C?
+L C_Small C16
 U 1 1 58B998EA
 P 8480 3575
-F 0 "C?" H 8490 3645 50  0000 L CNN
+F 0 "C16" H 8490 3645 50  0000 L CNN
 F 1 "10u" H 8490 3495 50  0000 L CNN
-F 2 "" H 8480 3575 50  0000 C CNN
+F 2 "Capacitors_SMD:C_0603" H 8480 3575 50  0001 C CNN
 F 3 "" H 8480 3575 50  0000 C CNN
 	1    8480 3575
@@
 $EndComp
 $Comp
-L C_Small C?
+L C_Small C17
 U 1 1 58B9A439
 P 8680 3580
-F 0 "C?" H 8690 3650 50  0000 L CNN
+F 0 "C17" H 8690 3650 50  0000 L CNN
 F 1 "100n" H 8690 3500 50  0000 L CNN
-F 2 "" H 8680 3580 50  0000 C CNN
+F 2 "Capacitors_SMD:C_0603" H 8680 3580 50  0001 C CNN
 F 3 "" H 8680 3580 50  0000 C CNN
 	1    8680 3580
@@
 $EndComp
 $Comp
-L ADS79XX U?
+L ADS79XX U4
 U 1 1 58B9BF2E
 P 7755 3405
-F 0 "U?" H 7305 4105 50  0000 L CNN
+F 0 "U4" H 7305 4105 50  0000 L CNN
 F 1 "ADS79XX" H 8055 4105 50  0000 C CNN
-F 2 "" H 7755 3405 50  0000 C CIN
+F 2 "Housings_DFN_QFN:QFN-16-1EP_3x3mm_Pitch0.5mm" H 7755 3405 50  0001 C CIN
 F 3 "" H 7755 3405 50  0000 C CNN
 	1    7755 3405
@@
 $EndComp
 $Comp
-L C_Small C?
+L C_Small C10
 U 1 1 58B851DB
 P 6805 3210
-F 0 "C?" H 6815 3280 50  0000 L CNN
+F 0 "C10" H 6815 3280 50  0000 L CNN
 F 1 "470p" H 6815 3130 50  0000 L CNN
-F 2 "" H 6805 3210 50  0000 C CNN
+F 2 "Capacitors_SMD:C_0603" H 6805 3210 50  0001 C CNN
 F 3 "" H 6805 3210 50  0000 C CNN
 	1    6805 3210
@@
 $EndComp
 $Comp
-L +3.3V #PWR?
+L +3.3V #PWR016
 U 1 1 58B9E7EB
 P 7755 1905
-F 0 "#PWR?" H 7755 1755 50  0001 C CNN
+F 0 "#PWR016" H 7755 1755 50  0001 C CNN
 F 1 "+3.3V" H 7755 2045 50  0000 C CNN
 F 2 "" H 7755 1905 50  0000 C CNN
@@
 $EndComp
 $Comp
-L C_Small C?
+L C_Small C15
 U 1 1 58B9E9E9
 P 7925 2530
-F 0 "C?" H 7935 2600 50  0000 L CNN
+F 0 "C15" H 7935 2600 50  0000 L CNN
 F 1 "1u" H 7935 2450 50  0000 L CNN
-F 2 "" H 7925 2530 50  0000 C CNN
+F 2 "Capacitors_SMD:C_0603" H 7925 2530 50  0001 C CNN
 F 3 "" H 7925 2530 50  0000 C CNN
 	1    7925 2530
@@
 $EndComp
 $Comp
-L GND #PWR?
+L GND #PWR017
 U 1 1 58B9F1E6
 P 8075 2530
-F 0 "#PWR?" H 8075 2280 50  0001 C CNN
+F 0 "#PWR017" H 8075 2280 50  0001 C CNN
 F 1 "GND" H 8075 2380 50  0000 C CNN
 F 2 "" H 8075 2530 50  0000 C CNN
@@
 $EndComp
 $Comp
-L GND #PWR?
+L GND #PWR018
 U 1 1 58BA0439
 P 8055 5350
-F 0 "#PWR?" H 8055 5100 50  0001 C CNN
+F 0 "#PWR018" H 8055 5100 50  0001 C CNN
 F 1 "GND" H 8055 5200 50  0000 C CNN
 F 2 "" H 8055 5350 50  0000 C CNN
@@
 $EndComp
 $Comp
-L C_Small C?
+L C_Small C13
 U 1 1 58BA0A88
 P 7040 4085
-F 0 "C?" H 7050 4155 50  0000 L CNN
+F 0 "C13" H 7050 4155 50  0000 L CNN
 F 1 "100n" H 7050 4005 50  0000 L CNN
-F 2 "" H 7040 4085 50  0000 C CNN
+F 2 "Capacitors_SMD:C_0603" H 7040 4085 50  0001 C CNN
 F 3 "" H 7040 4085 50  0000 C CNN
 	1    7040 4085
@@
 $EndComp
 $Comp
-L C_Small C?
+L C_Small C12
 U 1 1 58BA0B12
 P 6810 4090
-F 0 "C?" H 6820 4160 50  0000 L CNN
+F 0 "C12" H 6820 4160 50  0000 L CNN
 F 1 "1u" H 6820 4010 50  0000 L CNN
-F 2 "" H 6810 4090 50  0000 C CNN
+F 2 "Capacitors_SMD:C_0603" H 6810 4090 50  0001 C CNN
 F 3 "" H 6810 4090 50  0000 C CNN
 	1    6810 4090
@@
 $EndComp
 $Comp
-L R_Small R?
+L R_Small R10
 U 1 1 58BA14C3
 P 8675 3005
-F 0 "R?" H 8705 3025 50  0000 L CNN
+F 0 "R10" H 8705 3025 50  0000 L CNN
 F 1 "47" H 8705 2965 50  0000 L CNN
-F 2 "" H 8675 3005 50  0000 C CNN
+F 2 "Resistors_SMD:R_0603" H 8675 3005 50  0001 C CNN
 F 3 "" H 8675 3005 50  0000 C CNN
 	1    8675 3005
@@
 DVDD ? Wofür ? brauchen wir es?\nCH_SEL mit was gleichzeitig steuern ??\n
 $Comp
-L GND #PWR?
+L GND #PWR019
 U 1 1 58BA3940
 P 7130 3705
-F 0 "#PWR?" H 7130 3455 50  0001 C CNN
+F 0 "#PWR019" H 7130 3455 50  0001 C CNN
 F 1 "GND" H 7130 3555 50  0000 C CNN
 F 2 "" H 7130 3705 50  0000 C CNN
@@
 $EndComp
 $Comp
-L GND #PWR?
+L GND #PWR020
 U 1 1 58BA3B7B
 P 7655 2590
-F 0 "#PWR?" H 7655 2340 50  0001 C CNN
+F 0 "#PWR020" H 7655 2340 50  0001 C CNN
 F 1 "GND" H 7655 2440 50  0000 C CNN
 F 2 "" H 7655 2590 50  0000 C CNN
@@
 Connection ~ 7485 4960
 $Comp
-L GND #PWR?
+L GND #PWR021
 U 1 1 58C7E5F9
 P 7755 4270
-F 0 "#PWR?" H 7755 4020 50  0001 C CNN
+F 0 "#PWR021" H 7755 4020 50  0001 C CNN
 F 1 "GND" H 7755 4120 50  0000 C CNN
 F 2 "" H 7755 4270 50  0000 C CNN

Commit message: All parts in places (exept :Leds)
Connections:
- net ADC_1 renamed OpAmp_Out4
- net ADC_2 renamed OpAmp_Out2
Changed lines of the file:
@@
 $EndDescr
 Text GLabel 6345 3745 0    60   Input ~ 0
-ADC_1
+OpAmp_Out4
 Text GLabel 6335 3015 0    60   Input ~ 0
-ADC_2
+OpAmp_Out2
 $Comp
 L R_Small R5
