File: Test_Board_MKE14F256.sch (KiCad schematic (older format))
At the start: 0 parts

Commit message: v1.0
Changed lines of the file:
@@
 LIBS:ads7947X
 LIBS:ADS7944
+LIBS:NCP700B
+LIBS:mke14f256
+LIBS:mh-diodes
 EELAYER 25 0
 EELAYER END
 $Descr A3 16535 11693
 encoding utf-8
-Sheet 1 3
+Sheet 1 5
 Title "Test_Board_MKE14F"
 Date ""
@@
 F1 "ADC & REF.sch" 60
 $EndSheet
+$Sheet
+S 3715 9905 1185 825
+U 58BDE6CF
+F0 "OPAMP" 60
+F1 "OPAMP.sch" 60
+$EndSheet
+$Sheet
+S 4950 9910 1205 825
+U 58BD5D77
+F0 "mcu" 60
+F1 "mcu.sch" 60
+$EndSheet
 $EndSCHEMATC

Commit message: changed usd slot
Parts:
- added CON?: SD_Card, 10067847-001, symbol SD_Card
Changed lines of the file:
@@
 F1 "mcu.sch" 60
 $EndSheet
+$Comp
+L SD_Card CON?
+U 1 1 58D38F6D
+P 7550 3805
+F 0 "CON?" H 6900 4355 50  0000 C CNN
+F 1 "SD_Card" H 8150 3255 50  0000 C CNN
+F 2 "10067847-001" H 7750 4155 50  0000 C CNN
+F 3 "" H 7550 3805 50  0000 C CNN
+	1    7550 3805
+	1    0    0    -1
+$EndComp
 $EndSCHEMATC

Commit message: All parts in places (exept :Leds)
Parts:
- removed CON?: SD_Card, 10067847-001, symbol SD_Card
Changed lines of the file:
@@
 F1 "mcu.sch" 60
 $EndSheet
-$Comp
-L SD_Card CON?
-U 1 1 58D38F6D
-P 7550 3805
-F 0 "CON?" H 6900 4355 50  0000 C CNN
-F 1 "SD_Card" H 8150 3255 50  0000 C CNN
-F 2 "10067847-001" H 7750 4155 50  0000 C CNN
-F 3 "" H 7550 3805 50  0000 C CNN
-	1    7550 3805
-	1    0    0    -1
-$EndComp
 $EndSCHEMATC
