File: mcu.sch (KiCad schematic (older format))
At the start: 55 parts, among them P10 CONN_01X01, P11 CONN_01X01, P12 CONN_01X01, P13 CONN_01X01, P14 CONN_01X01, P15 CONN_01X01, P16 CONN_01X01, P17 CONN_01X01, P18 CONN_01X01, P19 CONN_01X01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

Commit message: Fixed some DRC errors
Parts:
- Y1: symbol QUARTZCMS4 -> QUARTZCMS4_(new)
Connections:
- wire segments 138 -> 141
Other:
- moved on the sheet: C27

Commit message: Complete... Still some things to check
Parts:
- D3, D4, D5, D6: symbol LED -> LED-RESCUE-Test_Board_MKE14F256
Changed lines of the file:
@@
 EESchema Schematic File Version 2
+LIBS:Test_Board_MKE14F256-rescue
 LIBS:power
 LIBS:device
@@
 $EndComp
 $Comp
-L LED D3
+L LED-RESCUE-Test_Board_MKE14F256 D3
 U 1 1 576313DE
 P 1622 10413
+AR Path="/576313DE" Ref="D3"  Part="1"
+AR Path="/58BD5D77/576313DE" Ref="D3"  Part="1"
 F 0 "D3" H 1622 10513 50  0000 C CNN
 F 1 "red" H 1622 10313 50  0000 C CNN
@@
 $EndComp
 $Comp
-L LED D4
+L LED-RESCUE-Test_Board_MKE14F256 D4
 U 1 1 576316C4
 P 1972 10413
+AR Path="/576316C4" Ref="D4"  Part="1"
+AR Path="/58BD5D77/576316C4" Ref="D4"  Part="1"
 F 0 "D4" H 1972 10513 50  0000 C CNN
 F 1 "yel" H 1972 10313 50  0000 C CNN
@@
 $EndComp
 $Comp
-L LED D5
+L LED-RESCUE-Test_Board_MKE14F256 D5
 U 1 1 57631F8D
 P 2272 10413
+AR Path="/57631F8D" Ref="D5"  Part="1"
+AR Path="/58BD5D77/57631F8D" Ref="D5"  Part="1"
 F 0 "D5" H 2272 10513 50  0000 C CNN
 F 1 "grn" H 2272 10313 50  0000 C CNN
@@
 $EndComp
 $Comp
-L LED D6
+L LED-RESCUE-Test_Board_MKE14F256 D6
 U 1 1 576325CC
 P 2572 10413
+AR Path="/576325CC" Ref="D6"  Part="1"
+AR Path="/58BD5D77/576325CC" Ref="D6"  Part="1"
 F 0 "D6" H 2572 10513 50  0000 C CNN
 F 1 "ble" H 2572 10313 50  0000 C CNN

Commit message: corrected some mistakes listed in the email
Parts:
- added R33: 5, Resistors_SMD:R_0603, symbol R_Small
- P4: value CONN_01X04 -> CONN_01X06; footprint Connectors_Molex:Molex_KK-6410-04_04x2.54mm_Straight -> Connectors_Molex:Molex_KK-6410-06_06x2.54mm_Straight; symbol CONN_01X04 -> CONN_01X06
Connections:
- net +3V3: now also R33.1; no longer C30.2, U7.8 (VDDA)
- net GND: now also P4.5 (P5), P4.6 (P6)
- new net: C30.2, R33.2, U7.8 (VDDA)
Other:
- note added: "die restlichen 2 pins ?!"

Commit message: V1.0
Parts:
- P4: Mnfr (none) -> 22-27-2061
- XS1: Manf ebay -> (none)
Connections:
- net +3V3: now also P4.1 (P1)
- net ADC_SPI1_CS0: no longer P4.3 (P3)
- net ADC_SPI1_MOSI_ADC_CH_SEL: now also P4.5 (P5); no longer P4.4 (P4)
- net ADC_SPI1_SCLK: now also P4.2 (P2); no longer P4.1 (P1)
- net ADC_SPI1_SDO: now also P4.3 (P3); no longer P4.2 (P2)
- net GND: no longer P4.5 (P5)
- net ADC_SPI1_CS1: now reaches U7.38 (PTA6)
- net ADC_SPI1_CS1: now also P4.4 (P4)
Other:
- note removed: "die restlichen 2 pins ?!"
